Commit message: trying something out, wish me luck

File: dummy_description/model/robot.urdf (robot description, URDF)
Before this commit: robot dummy, 11 links, 10 joints
Links:
- removed link base
- link arm_round: mass 0.00045359236800000010507 -> 0.00045359236799999999665
- link arm_round_2: mass 0.00045359236800000010507 -> 0.00045359236799999999665
- link arm_round_3: mass 0.00045359236800000010507 -> 0.00045359236799999999665
- link mg996r_v2: mass 0.055791861264000007503 -> 0.1120373148959999815; geometry collision mesh filename=package://dummy_description/model/arm_round.stl; collision mesh filename=package://dummy_description/model/composite_part_1.stl
- link mg996r_v2_2: mass 0.055791861264000007503 -> 0.055791861263999993625
- link mg996r_v2_3: mass 0.055791861264000007503 -> 0.055791861263999993625
- link seg_one: mass 0.038138749034982870334 -> 0.037612434876134324957
- link seg_two: mass 0.030280862737785154554 -> 0.029688462028335853293
- link wrist: mass 0.016076987416131532926 -> 0.015756700876425590307
Joints:
- removed joint shoulder_servo
- joint base_link_to_base: child base -> mg996r_v2
- joint elbow: origin xyz=-0.014461892066012130287 -0.0050000032706329772259 -0.015500000000000027645 rpy=-3.141592653589793116 1.1221675757108101127e-15 -1.5707963267949012209 -> xyz=-0.014461892066012116409 -0.0050000032706329911036 -0.0154999999999996807 rpy=-3.141592653589793116 -1.1146035864132190215e-15 -1.5707963267949107689
- joint elbow_servo: origin xyz=0.125 -0.041750000000000023204 0 rpy=3.141592653589793116 -0 -1.570796326794896558 -> xyz=0.125 -0.041750000000000023204 0 rpy=-3.1415926535897926719 -1.5256280989911611756e-17 -1.570796326794896558
- joint forearm_mount: origin xyz=6.9388939039072283776e-17 -0.0072000000000007752243 0.0018999999999999919731 rpy=-3.1415926535897926719 2.3408220465313534229e-16 -1.0587911840678691044e-20 -> xyz=5.5511151231257827021e-17 -0.0072000000000007752243 0.0018999999999999850342 rpy=-3.1415926535897926719 -3.1918273395219628395e-16 2.9490299091605492575e-17
- joint shoulder: origin xyz=-0.01446189206601210947 0.0049999967293670455337 -0.015499999999999999889 rpy=3.141592653589793116 2.8943195551387177825e-16 1.570796326794891673 -> xyz=-0.060670203732602304147 -0.078408841567689263607 0.049027741493738577483 rpy=1.5707964286944553489 -0.012215162504253881601 6.0580177925737935818e-08
- joint shoulder_horn: origin xyz=5.5511151231257827021e-17 0.0071999999999992347899 0.0019000000000000127898 rpy=-3.1415926535897922278 -1.0323879464612367862e-23 -2.7724023638343179296e-17 -> xyz=5.5511151231257827021e-17 0.0071999999999992347899 0.0019000000000000127898 rpy=-3.1415926535897922278 -1.6029012262867187634e-15 -4.1633363423442630709e-17
- joint wrist: origin xyz=0.034538107933987892417 -0.0050000032706329633481 -0.015499999999999986011 rpy=-3.1415926535897922278 -6.1232673501503056481e-17 -1.5707963267948907848 -> xyz=0.034538107933987885478 -0.0050000032706329911036 -0.015499999999999750089 rpy=-3.1415926535897895633 7.6639611212484526416e-16 -1.57079632679489678
- joint wrist_mount: origin xyz=4.1633363423443370266e-17 0.0071999999999992347899 0.0018999999999999850342 rpy=3.141592653589793116 1.9249019073327577723e-15 -7.4941282359972137417e-16 -> xyz=5.5511151231257827021e-17 0.0071999999999992486677 0.0019000000000000266676 rpy=3.1415926535897922278 1.9398011109958429029e-15 -7.7195194680968487625e-16
- joint wrist_servo: origin xyz=-0.099000000000000004663 -0.0022500000000000019984 6.9388939039072283776e-18 rpy=-3.1415926535897926719 6.3475081490357335169e-16 3.141592653589793116 -> xyz=-0.098999999999999990785 -0.0022500000000000019984 1.3877787807814456755e-17 rpy=-3.1415926535897926719 2.2409496976941053526e-16 -3.141592653589793116

Commit message: updated urdf I think

File: dummy_description/model/robot.urdf (robot description, URDF)
Before this commit: robot dummy, 10 links, 9 joints
Links:
- added link arm_round_4, mass 0.00045359236799999999665; collision mesh filename=package://dummy_description/model/arm_round.stl; visual mesh filename=package://dummy_description/model/arm_round.stl
- added link base, mass 0; collision mesh filename=package://dummy_description/model/base.stl; visual mesh filename=package://dummy_description/model/base.stl
- added link ee, mass 0; collision mesh filename=package://dummy_description/model/ee.stl; visual mesh filename=package://dummy_description/model/ee.stl
- added link final-2-arms-horn, mass 0; collision mesh filename=package://dummy_description/model/final-2-arms-horn.stl; visual mesh filename=package://dummy_description/model/final-2-arms-horn.stl
- added link mg996r_v2_4, mass 0.055791861264000007503; collision mesh filename=package://dummy_description/model/mg996r_v2.stl; visual mesh filename=package://dummy_description/model/mg996r_v2.stl
- added link part_1, mass 0; collision mesh filename=package://dummy_description/model/part_1.stl; visual mesh filename=package://dummy_description/model/part_1.stl
- added link servo-sg90-final, mass 0; collision mesh filename=package://dummy_description/model/servo-sg90-final.stl; visual mesh filename=package://dummy_description/model/servo-sg90-final.stl
- link mg996r_v2: mass 0.1120373148959999815 -> 0.055791861264000007503; geometry collision mesh filename=package://dummy_description/model/mg996r_v2.stl; visual mesh filename=package://dummy_description/model/mg996r_v2.stl
- link mg996r_v2_2: mass 0.055791861263999993625 -> 0.055791861264000007503
- link mg996r_v2_3: mass 0.055791861263999993625 -> 0.055791861264000007503
- link seg_one: mass 0.037612434876134324957 -> 0.037612434876134331896
- link seg_two: mass 0.029688462028335853293 -> 0.029688462028335856763
Joints:
- added joint ee: type fixed, parent final-2-arms-horn, child ee, origin xyz=-0.0050000000000000044409 6.9388939039072283776e-18 -0.0020000000000000156541 rpy=2.0816681711721675888e-17 3.5182360497154520276e-17 -8.5796560150450912835e-16, axis 0 0 1, limit effort=1 velocity=20
- added joint joint: type fixed, parent arm_round, child part_1, origin xyz=4.1633363423443370266e-17 4.1633363423443370266e-17 0.0019000000000000058509 rpy=-3.141592653589793116 7.0439937520025449219e-16 -1.570796326794896558, axis 0 0 1, limit effort=1 velocity=20
- added joint servo_joint: type fixed, parent base, child mg996r_v2, origin xyz=-0.028538075398620611767 -0.060918143323766021924 -0.062985219167393094453 rpy=3.141571259400607552 1.2221860805481506306e-06 -1.4862894919532512592e-06, axis 0 0 1, limit effort=1 velocity=20
- added joint shoulder_joint: type fixed, parent part_1, child mg996r_v2_2, origin xyz=-0.0039999999999999688582 0.0050000000000000113798 -0.065749999999999989009 rpy=-3.141592653589793116 1.570796326794896558 0, axis 0 0 1, limit effort=1 velocity=20
- added joint torso: type revolute, parent mg996r_v2, child arm_round, origin xyz=-0.01446189206601211294 -0.0050000032706329772259 -0.01549999999999999295 rpy=-3.141592653589793116 -5.8824087670381847472e-16 -0.00060706039085584560539, axis 0 0 1, limit lower=-2.356194490192344837 upper=0.785398163397448279 effort=1 velocity=20
- added joint wristr: type revolute, parent servo-sg90-final, child final-2-arms-horn, origin xyz=6.9388939039072283776e-18 0.0082499999999999934497 -0.013999999999999998557 rpy=1.2004286453759497205e-15 -6.8497860378561265184e-17 -1.5707963207310067233, axis 0 0 1, limit lower=0 upper=3.141592653589793116 effort=1 velocity=20
- added joint wristr_mount: type fixed, parent wrist, child servo-sg90-final, origin xyz=-0.039999999999999980016 0.0072500000000000064393 0.034000000000000009381 rpy=-1.570796326794896558 -5.8966664491229107969e-16 -1.570796326794896558, axis 0 0 1, limit effort=1 velocity=20
- joint base_link_to_base: child mg996r_v2 -> base
- joint elbow: child arm_round_2 -> arm_round_3; origin xyz=-0.014461892066012116409 -0.0050000032706329911036 -0.0154999999999996807 rpy=-3.141592653589793116 -1.1146035864132190215e-15 -1.5707963267949107689 -> xyz=-0.014461892066012123348 -0.0050000032706329772259 -0.01549999999999999295 rpy=-3.141592653589793116 -2.8072184884609522565e-15 -1.5707963267949354158; parent mg996r_v2_2 -> mg996r_v2_3
- joint elbow_servo: child mg996r_v2_2 -> mg996r_v2_3; origin xyz=0.125 -0.041750000000000023204 0 rpy=-3.1415926535897926719 -1.5256280989911611756e-17 -1.570796326794896558 -> xyz=0.125 -0.041750000000000016265 0 rpy=-3.1415926535897913396 -1.0939599920378727413e-16 -1.570796326794896558
- joint forearm_mount: origin xyz=5.5511151231257827021e-17 -0.0072000000000007752243 0.0018999999999999850342 rpy=-3.1415926535897926719 -3.1918273395219628395e-16 2.9490299091605492575e-17 -> xyz=5.5511151231257827021e-17 -0.0072000000000007613465 0.0018999999999999919731 rpy=-3.1415926535897926719 -6.6629369224388344028e-16 0; parent arm_round_2 -> arm_round_3
- joint shoulder: child arm_round -> arm_round_2; origin xyz=-0.060670203732602304147 -0.078408841567689263607 0.049027741493738577483 rpy=1.5707964286944553489 -0.012215162504253881601 6.0580177925737935818e-08 -> xyz=-0.01446189206601211294 0.0049999967293670177781 -0.015499999999999979072 rpy=3.1415926535897926719 -4.5286110422765151629e-15 1.5367034096982505886; parent mg996r_v2 -> mg996r_v2_2
- joint shoulder_horn: origin xyz=5.5511151231257827021e-17 0.0071999999999992347899 0.0019000000000000127898 rpy=-3.1415926535897922278 -1.6029012262867187634e-15 -4.1633363423442630709e-17 -> xyz=4.8572257327350598644e-17 0.0071999999999992417288 0.001899999999999998912 rpy=-3.1415926535897917837 4.1494132382737779046e-17 5.5511151231256939553e-17; parent arm_round -> arm_round_2
- joint wrist: child arm_round_3 -> arm_round_4; origin xyz=0.034538107933987885478 -0.0050000032706329911036 -0.015499999999999750089 rpy=-3.1415926535897895633 7.6639611212484526416e-16 -1.57079632679489678 -> xyz=0.034538107933987871601 -0.0050000032706329772259 -0.01549999999999999295 rpy=-3.1415926535897855665 8.3616720860691773698e-16 -1.5707963267948976682; parent mg996r_v2_3 -> mg996r_v2_4
- joint wrist_mount: origin xyz=5.5511151231257827021e-17 0.0071999999999992486677 0.0019000000000000266676 rpy=3.1415926535897922278 1.9398011109958429029e-15 -7.7195194680968487625e-16 -> xyz=4.1633363423443370266e-17 0.0071999999999992347899 0.0019000000000000266676 rpy=3.141592653589793116 1.9587128685487484756e-15 -7.8409501114152252592e-16; parent arm_round_3 -> arm_round_4
- joint wrist_servo: child mg996r_v2_3 -> mg996r_v2_4; origin xyz=-0.098999999999999990785 -0.0022500000000000019984 1.3877787807814456755e-17 rpy=-3.1415926535897926719 2.2409496976941053526e-16 -3.141592653589793116 -> xyz=-0.099000000000000018541 -0.0022499999999999881206 0 rpy=-3.1415926535897926719 5.0856376960828415199e-16 -3.141592653589793116
